File: ADC.sch (KiCad schematic (older format))
At the start: 17 parts, among them J10 TBL009-254-02GY-2GY, J3 TBL009-254-02GY-2GY, J4 TBL009-254-02GY-2GY, J5 TBL009-254-02GY-2GY, J6 TBL009-254-02GY-2GY, J7 TBL009-254-02GY-2GY, J8 TBL009-254-02GY-2GY, J9 TBL009-254-02GY-2GY, U5 MCP3008

Commit message: Rev1.1
Mostly as Orderd, some small none function changes to Rev1
Parts:
- J10, J3, J4, J6, J7, J8, J9: symbol SamacSys_Parts:TBL009-254-02GY-2GY -> Samacsys:TBL009-254-02GY-2GY
- J5: footprint SamacSys_Parts:TBL00925402GY2GY -> TBL00925402GY2GY; symbol SamacSys_Parts:TBL009-254-02GY-2GY -> Samacsys:TBL009-254-02GY-2GY; Mouser Price/Stock (none) -> https://www.mouser.co.uk/ProductDetail/CUI-Devices/TBL009-2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
Changed lines of the file:
@@
 $Descr A4 11693 8268
 encoding utf-8
-Sheet 2 2
+Sheet 2 3
 Title "Snapmaker2 CANbus extension"
 Date "2021-01-16"
@@
 Ambient
 $Comp
-L SamacSys_Parts:TBL009-254-02GY-2GY J3
+L Samacsys:TBL009-254-02GY-2GY J3
 U 1 1 6006A4CD
 P 3600 1900
@@
 Connection ~ 4850 1800
 $Comp
-L SamacSys_Parts:TBL009-254-02GY-2GY J4
+L Samacsys:TBL009-254-02GY-2GY J4
 U 1 1 60089421
 P 3600 2300
@@
 $EndComp
 $Comp
-L SamacSys_Parts:TBL009-254-02GY-2GY J5
+L Samacsys:TBL009-254-02GY-2GY J5
 U 1 1 600898E9
 P 3600 2700
 F 0 "J5" H 4000 2335 50  0000 C CNN
 F 1 "TBL009-254-02GY-2GY" H 4000 2426 50  0000 C CNN
-F 2 "SamacSys_Parts:TBL00925402GY2GY" H 4250 2800 50  0001 L CNN
+F 2 "TBL00925402GY2GY" H 4250 2800 50  0001 L CNN
 F 3 "https://componentsearchengine.com/Datasheets/1/TBL009-254-02GY-2GY.pdf" H 4250 2700 50  0001 L CNN
 F 4 "Fixed Terminal Blocks Terminal block, screwless, 2.54, Horizontal, 2, Gray w Gray Button" H 4250 2600 50  0001 L CNN "Description"
 F 5 "10.5" H 4250 2500 50  0001 L CNN "Height"
 F 6 "490-TBL00925402GY2GY" H 4250 2400 50  0001 L CNN "Mouser Part Number"
-F 7 "" H 4250 2300 50  0001 L CNN "Mouser Price/Stock"
+F 7 "https://www.mouser.co.uk/ProductDetail/CUI-Devices/TBL009-254-02GY-2GY/?qs=UXgszm6BlbEjVz5a2Fsubg%3D%3D" H 4250 2300 50  0001 L CNN "Mouser Price/Stock"
 F 8 "CUI Devices" H 4250 2200 50  0001 L CNN "Manufacturer_Name"
 F 9 "TBL009-254-02GY-2GY" H 4250 2100 50  0001 L CNN "Manufacturer_Part_Number"
@@
 $EndComp
 $Comp
-L SamacSys_Parts:TBL009-254-02GY-2GY J6
+L Samacsys:TBL009-254-02GY-2GY J6
 U 1 1 6008A026
 P 3600 3100
@@
 $EndComp
 $Comp
-L SamacSys_Parts:TBL009-254-02GY-2GY J7
+L Samacsys:TBL009-254-02GY-2GY J7
 U 1 1 6008A72C
 P 3600 3500
@@
 $EndComp
 $Comp
-L SamacSys_Parts:TBL009-254-02GY-2GY J8
+L Samacsys:TBL009-254-02GY-2GY J8
 U 1 1 6008AF27
 P 3600 3900
@@
 $EndComp
 $Comp
-L SamacSys_Parts:TBL009-254-02GY-2GY J9
+L Samacsys:TBL009-254-02GY-2GY J9
 U 1 1 6008B333
 P 3600 4300
@@
 $EndComp
 $Comp
-L SamacSys_Parts:TBL009-254-02GY-2GY J10
+L Samacsys:TBL009-254-02GY-2GY J10
 U 1 1 6008B85A
 P 3600 4700

Commit message: Rev2 done
Orderd and Assembeld PCB, works sofar, no magic Smoke sofar :D
Parts:
- removed J3: TBL009-254-02GY-2GY, SamacSys_Parts:TBL00925402GY2GY, symbol Samacsys:TBL009-254-02GY-2GY
- added J15: DB9_Female_MountingHoles, SamacSys_Parts:D09S23A4GV00LF, symbol Connector:DB9_Female_MountingHoles
- added J17: TBL009-254-02GY-2GY, SamacSys_Parts:TBL00925402GY2GY, symbol Samacsys:TBL009-254-02GY-2GY
- added J3: DB9_Male_MountingHoles, SamacSys_Parts:D09P23A4GV00LF, symbol Connector:DB9_Male_MountingHoles
- J5: footprint TBL00925402GY2GY -> SamacSys_Parts:TBL00925402GY2GY; Mouser Price/Stock https://www.mouser.co.uk/ProductDetail/CUI-Devices/TBL009-2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 -> (none)
- R10, R9: value Res -> 27k; Mouser Part Number (none) -> 71-CRCW1206-27K-E3
Connections:
- net GND: now also J10.1, J10.2, J4.1, J4.2, J5.1, J5.2, J6.1, J6.2, J7.1, J7.2, J8.1, J8.2, J9.1, J9.2, J15.0 (PAD), J15.5, J17.1, J17.2, J3.0 (PAD), J3.5; no longer J10.3, J10.4, J4.3, J4.4, J5.3, J5.4, J6.3, J6.4, J7.3, J7.4, J8.3, J8.4, J9.3, J9.4
- net at R3.2, U5.1 (CH0): now also J15.9
- net at R4.2, U5.2 (CH1): now also J15.4; no longer J4.1, J4.2
- net at R5.2, U5.3 (CH2): now also J15.8; no longer J5.1, J5.2
- net at R6.2, U5.4 (CH3): now also J15.3; no longer J6.1, J6.2
- net at R7.2, U5.5 (CH4): now also J15.7; no longer J7.1, J7.2
- net at R8.2, U5.6 (CH5): now also J15.2; no longer J8.1, J8.2
- net at R9.2, U5.7 (CH6): now also J15.6; no longer J9.1, J9.2
- net at R10.2, U5.8 (CH7): now also J15.1; no longer J10.1, J10.2
- new net: J17.3, J17.4, J3.1
- new net: J3.2, J9.3, J9.4
- new net: J3.3, J7.3, J7.4
- new net: J3.4, J5.3, J5.4
- new net: J10.3, J10.4, J3.6
- new net: J3.7, J8.3, J8.4
- new net: J3.8, J6.3, J6.4
- new net: J3.9, J4.3, J4.4
