File: SNModule.sch (KiCad schematic (older format))
At the start: 52 parts, among them J1 DB9_Male_MountingHoles, J11 Conn_01x04, J12 Conn_01x04, J13 Conn_01x04, J14 Conn_01x02, J2 DB9_Female_MountingHoles, Q1 KSC1815, SW2 SW_Push, SW3 SW_Push, U1 Teensy4.0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

Commit message: Rev1
Orderd and ariving soon
Parts:
- removed C5: 0.1uF, Capacitors_SMD:C_1206_HandSoldering, symbol Device:C_Small
- added C5: 100uF, Capacitors_SMD:CP_Elec_6.3x7.7, symbol Device:C
- D2, D3, D4: Manufacturer_Name (none) -> Lite-On; Manufacturer_Part_Number (none) -> LTL-307GE; Mouser Part Number (none) -> 859-LTL-307GE
- J11, J12, J13: Manufacturer_Name (none) -> Samtec; Manufacturer_Part_Number (none) -> SLW-104-01-T-S; Mouser Part Number (none) -> 200-SLW10401TS
- J14: Manufacturer_Name (none) -> Samtec; Manufacturer_Part_Number (none) -> SLW-102-01-T-S; Mouser Part Number (none) -> 200-SLW10201TS
- J2: Mouser Part Number 649-D09S23A4GV00LF -> 649-D09S23A4GV00LF
- JP1: Manufacturer_Name (none) -> Kycon; Manufacturer_Part_Number (none) -> SX1100-B; Mouser Part Number (none) -> 806-SX1100-B
- Q1: Manufacturer_Name (none) -> ON Semiconductor / Fairchild; Manufacturer_Part_Number (none) -> KSC1815YTA; Mouser Part Number (none) -> 512-KSC1815YTA
Connections:
- wire segments 222 -> 224
Other:
- note added: "Alternative to JP1, Costs more though\n611-SPA02B SIP Toggle switch\n"
- note added: "For JP1, you'll need a 2x1, 2.54mm Header strip\nKICAD BOM has only Jumper, Mouser BOM has them seperatly."
- moved on the sheet: C6, C7, C8, C9, D5, J2, JP1, R14, U3

Commit message: Rev1.1
Mostly as Orderd, some small none function changes to Rev1
Parts:
- U1: symbol Teensy_Component:Teensy4.0 -> Teensy:Teensy4.0
- U7: symbol SamacSys_Parts:EN11-HSM1AF15 -> Samacsys:EN11-HSM1AF15
Connections:
- wire segments 224 -> 225
Other:
- moved on the sheet: BZ1, FID1, FID2, FID3, H1, H2, H3, H4, J11, R15, R16, R17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

Commit message: Rev2 done
Orderd and Assembeld PCB, works sofar, no magic Smoke sofar :D
Parts:
- removed Q1: KSC1815, TO_SOT_Packages_THT:TO-92_Inline_Wide, symbol Transistor_BJT:2N3904
- added D6, D7: CDSOT23-T24CAN, TO_SOT_Packages_SMD:SOT-23, symbol SNModule-rescue:CDSOT23-T24CAN-Samacsys
- added H5, H6: MountingHole_Pad, Mounting_Holes:MountingHole_4.3mm_M4_Pad_Via, symbol Mechanical:MountingHole_Pad
- added J16: TBL009-254-02GY-2GY, SamacSys_Parts:TBL00925402GY2GY, symbol SNModule-rescue:TBL009-254-02GY-2GY-Samacsys
- added Q1: BC337, TO_SOT_Packages_THT:TO-92_Inline_Wide, symbol Transistor_BJT:BC337
- added R21, R22: 1M, Resistors_SMD:R_1206_HandSoldering, symbol Device:R_Small
- added R23: 120R, Resistors_SMD:R_1206_HandSoldering, symbol Device:R
- added U8: TLP785, Housings_DIP:DIP-4_W7.62mm_LongPads, symbol Isolator:TLP785
- BZ1: footprint Buzzers_Beepers:Buzzer_12x9.5RM7.6 -> Blanket Github additions:Buzzer_TDK_12.2x6.5RM5
- R14: Manufacturer_Part_Number CRCW1206120RFKEAC -> CRCW1206120RFKEAC
- U1: symbol Teensy:Teensy4.0 -> SNModule-rescue:Teensy4.0-Teensy
- U7: symbol Samacsys:EN11-HSM1AF15 -> SNModule-rescue:EN11-HSM1AF15-Samacsys
Connections:
- net +3V3: no longer SW2.1, SW3.1, U7.C1, U7.D1
- net +5V: now also R21.1
- net GND: now also SW2.1, SW3.1, U7.C1, U7.D1, D6.3 (K3), D7.3 (K3), H5.1, H6.1, Q1.3 (E), R21.2, R22.2, U8.2
- net Mod_CAN_N: now also D7.1 (K1)
- net Mod_CAN_P: now also D7.2 (K2)
- net SN_CAN_N: now also D6.2 (K2)
- net SN_CAN_P: now also D6.1 (K1)
- net Opto1: now reaches U1.7 (5_IN2)
- net Opto1: now also R23.2
- net at C5.1, D5.1 (K), J2.9: now also R22.1
- net at BZ1.2 (+), R19.1: now also Q1.1 (C)
- net at R20.1: now also Q1.2 (B)
- new net: R23.1, U8.1
- new net: J16.3, J16.4, U8.3
- new net: J16.1, J16.2, U8.4
- no-connect marks 42 -> 41
Other:
- note added: "Bottons, Rotaryencoder Inputs use internal PullUPs of Teensy"
- note added: "Optocoupler output"
- note removed: "Alternative to JP1, Costs more though\n611-SPA02B SIP Toggle switch\n"
- note removed: "Bottons, Rotaryencoder Inputs use internal Pulldowns of Teensy"
- moved on the sheet: BZ1, C5, D5, FID1, FID2, FID3, H1, H2, H3, H4, J1, R15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
